Commit message: modify urdf files
camera and ur3_robot_hri_hand files were changed for real robot environment

File: Ur_hrihand/ur_hrihand_gazebo/urdf/d435_camera_g.urdf.xacro (robot description, xacro)
@@ -10,5 +10,5 @@
   <!--<xacro:include filename="$(find realsense2_description)/urdf/_materials.urdf.xacro" />-->
   <xacro:include filename="$(find realsense2_description)/urdf/_usb_plug.urdf.xacro" />
-  <xacro:macro name="g_sensor_d435" params="parent *origin name:=g_camera use_nominal_extrinsics:=true">
+  <xacro:macro name="g_sensor_d435" params="parent *origin name:=camera use_nominal_extrinsics:=true"> <!--real_robot: camera/ simulation g_sensor_d435-->
     <xacro:arg name="add_plug" default="false" />
     <xacro:property name="M_PI" value="3.1415926535897931" />
@@ -134,6 +134,6 @@
       </xacro:usb_plug>
     </xacro:if>-->
-   <gazebo reference="g_camera_link">
-        <sensor type="depth" name="g_camera">
+   <gazebo reference="camera_link">
+        <sensor type="depth" name="camera">
             <always_on>1</always_on>
             <visualize>true</visualize>
@@ -155,9 +155,9 @@
                 <alwaysOn>true</alwaysOn>
                     <updateRate>20.0</updateRate>
-                    <cameraName>g_d435</cameraName>
-                    <frameName>g_camera_depth_optical_frame</frameName>
-                <imageTopicName>rgb/g_image_raw</imageTopicName>
-                <depthImageTopicName>depth/g_image_raw</depthImageTopicName>
-                <pointCloudTopicName>depth/g_points</pointCloudTopicName>
+                    <cameraName>camera</cameraName>
+                    <frameName>camera_depth_optical_frame</frameName>
+                <imageTopicName>rgb/image_raw</imageTopicName>
+                <depthImageTopicName>depth/image_raw</depthImageTopicName>
+                <pointCloudTopicName>depth/points</pointCloudTopicName>
                 <cameraInfoTopicName>rgb/camera_info</cameraInfoTopicName>
                 <depthImageCameraInfoTopicName>depth/camera_info</depthImageCameraInfoTopicName>

File: Ur_hrihand/ur_hrihand_gazebo/urdf/ur3_robot_hri_hand.urdf.xacro (robot description, xacro)
@@ -7,5 +7,4 @@
   <!-- ur3 -->
   <xacro:include filename="$(find ur_hrihand_gazebo)/urdf/ur3.urdf.xacro" />
-  <!-- <xacro:include filename="$(find ur_robot_server)/urdf/hri_hand.xacro" /> -->
   <xacro:include filename="$(find ur_hrihand_gazebo)/urdf/d435_camera_g.urdf.xacro" />
   <!-- arm -->
@@ -20,5 +19,5 @@
   />
   <xacro:g_sensor_d435 parent="gripper_link">
-    <origin xyz="-0.07 0.0 0.00" rpy="0 ${-pi/2} 0"/>
+    <origin xyz="-0.085 0.0 -0.03" rpy="0 ${-pi/2} 0"/>
   </xacro:g_sensor_d435>
   <!-- Configure self collision properties per link -->
